Commit message: fk and gui functioning

File: urdf/articulated.urdf (robot description, URDF)
Before this commit: robot articulated, 3 links, 2 joints
Links:
- removed link base
- removed link link1
- removed link link2
- added link joint1; visual mesh filename=file:///$(find articulated)/meshes/link1.dae
- added link joint2; visual mesh filename=file:///$(find articulated)/meshes/link2.dae
- added link slide; visual mesh filename=file:///$(find articulated)/meshes/base.dae
Joints:
- joint j1: child link1 -> joint1; parent base -> slide
- joint j2: child link2 -> joint2; parent link1 -> joint1
